File: hw/motor_driver/half_bridge.kicad_sch (KiCad schematic)
At the start: 5 parts, among them Q1 Q_NIGBT_GCE, Q2 Q_NIGBT_GCE, U2 L6388

Commit message: finished PCB
Connections:
- net OUT: now also U2.6 (OUT); no longer U2.12 (OUT)
Changed lines of the file:
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@@
     )
     (pin "1")
-    (pin "12")
     (pin "2")
     (pin "3")
     (pin "4")
     (pin "5")
+    (pin "6")
     (pin "7")
     (pin "8")
