File: hw/motor_driver/motor_driver.kicad_sch (KiCad schematic)
At the start: 37 parts, among them J1 Conn_01x03_Socket, J2 MOTOR, Q7 NPN, T1 Transformer_1P_1S, U3 LM317_TO-220, U4 TODO, U7 STM32G030K6Tx

Commit message: finished PCB
Parts:
- removed Q7: NPN, symbol Simulation_SPICE:NPN
- added C10: 100n, Capacitor_SMD:C_0603_1608Metric_Pad1.08x0.95mm_HandSolder, symbol Device:C
- added D4: LED_Filled, LED_THT:LED_D5.0mm, symbol Device:LED_Filled
- added H1, H2, H3, H4: MountingHole, MountingHole:MountingHole_3.2mm_M3, symbol Mechanical:MountingHole
- added HS2: Heatsink_Pad, myLib:heatsink_56x58, symbol Mechanical:Heatsink_Pad
- added J3: Conn_01x04_Pin, Connector_PinHeader_2.54mm:PinHeader_1x04_P2.54mm_Vertical, symbol Connector:Conn_01x04_Pin
- added J5: SWD, Connector_PinHeader_2.54mm:PinHeader_1x04_P2.54mm_Vertical, symbol Connector:Conn_01x04_Pin
- added NT1: NetTie_2, NetTie:NetTie-2_SMD_Pad2.0mm, symbol Device:NetTie_2
- added R14, R15, R16: R, Resistor_SMD:R_0603_1608Metric_Pad0.98x0.95mm_HandSolder, symbol Device:R
- added RV2: Varistor, Varistor:RV_Disc_D15.5mm_W4.9mm_P7.5mm, symbol Device:Varistor
- added U8, U9: SFH617A-1X007T, Package_DIP:SMDIP-4_W9.53mm_Clearance8mm, symbol Isolator:SFH617A-1X007T
- C101: value C -> 0.1u; footprint Capacitor_SMD:C_0603_1608Metric_Pad1.08x0.95mm_HandSolder -> Capacitor_THT:C_Rect_L19.0mm_W6.0mm_P15.00mm_MKS4
- C2, C3: value C -> 4.7n; footprint Capacitor_SMD:C_0603_1608Metric_Pad1.08x0.95mm_HandSolder -> Capacitor_THT:C_Rect_L13.0mm_W6.0mm_P10.00mm_FKS3_FKP3_MKS4
- D1: footprint Diode_THT:Diode_Bridge_19.0x3.5x10.0mm_P5.0mm -> Diode_THT:Diode_Bridge_Vishay_KBL
- D2: value D_Bridge_-AA+ -> D_Bridge_+A-A; footprint Diode_THT:Diode_Bridge_Round_D9.0mm -> Diode_THT:Diode_Bridge_19.0x3.5x10.0mm_P5.0mm; symbol Device:D_Bridge_-AA+ -> Device:D_Bridge_-A+A
- D3: footprint (none) -> Diode_SMD:D_MiniMELF_Handsoldering
- FL1: footprint (none) -> Inductor_THT:L_CommonMode_Toroid_Vertical_L38.1mm_W20.3mm_Px15.24mm_Py22.86mm_Bourns_8100
- J1: value Conn_01x03_Socket -> PWR IN
- J2: footprint (none) -> TerminalBlock_Phoenix:TerminalBlock_Phoenix_MKDS-1,5-3-5.08_1x03_P5.08mm_Horizontal
- L1: footprint (none) -> myLib:Coil_40x48
- R13: value 3k3 -> R
- R3, R4: footprint Resistor_SMD:R_0603_1608Metric_Pad0.98x0.95mm_HandSolder -> Resistor_THT:R_Axial_DIN0411_L9.9mm_D3.6mm_P12.70mm_Horizontal
- U4: value TODO -> MCP6006; footprint Package_TO_SOT_SMD:TSOT-23-5 -> Package_TO_SOT_SMD:TSOT-23-5_HandSoldering
Connections:
- net +12V: now also D2.3 (+); no longer D2.4 (+)
- net +3.3V: now also R12.1, C10.2, J5.1 (Pin_1), R14.1, R15.1
- net DC_bus+: now also HS2.1; no longer R12.1
- net DC_bus_voltage: now also U7.17 (PB2); no longer U7.11 (PA4)
- net Earth: now also J1.2 (Pin_2); no longer J1.3 (Pin_3)
- net GND: now also C10.1, D4.1 (K), J5.4 (Pin_4), NT1.2, U9.3; no longer R5.2, R7.1
- net LINE: now also F1.2, T1.2 (AB), TH1.2; no longer F1.1, J1.1 (Pin_1), T1.1 (AA)
- net NEUT: now also FL1.4, J1.1 (Pin_1), T1.1 (AA); no longer FL1.3, J1.2 (Pin_2), T1.2 (AB)
- net drive_U_N: now also U7.28 (PB4); no longer U7.14 (PA7)
- net drive_U_P: now also U7.27 (PB3); no longer U7.18 (PA8)
- net drive_V_N: now also U7.30 (PB6); no longer U7.15 (PB0)
- net drive_V_P: now also U7.29 (PB5); no longer U7.19 (PA9/NC)
- net drive_W_N: now also U7.32 (PB8); no longer U7.16 (PB1)
- net drive_W_P: now also U7.31 (PB7); no longer U7.21 (PA10/NC)
- net shunt-: now reaches C4.2, D1.1 (-), R5.1, R6.1
- net at C101.1, FL1.2: now also D1.3, RV2.1; no longer TH1.2
- net at C2.1, FL1.1: now also TH1.1; no longer F1.2
- net at R12.2: now also D4.2 (A)
- net at D1.2, L1.2: now also RV2.2
- net at D2.2: now also T1.3 (SA); no longer T1.4 (SB)
- net at R13.2: now also J3.3 (Pin_3), U8.4
- net at L1.1: now also C101.2, FL1.3; no longer TH1.1
- net at RV1.2: now also U7.15 (PB0); no longer U7.31 (PB7)
- net SWCLK: now reaches U7.25 (PA14)
- net SWCLK: now also J5.3 (Pin_3)
- net brake: no longer names the net of R13.1
- net brake: now also J3.1 (Pin_1), R16.2; no longer U7.24 (PA13)
- new net: R14.2, U8.1
- new net: J3.4 (Pin_4), U8.3
- new net: J3.2 (Pin_2), U9.2
- new net: R16.1, U9.1
- new net: D2.4, T1.4 (SB)
- new net: F1.1, J1.3 (Pin_3)
- new net SWDIO: J5.2 (Pin_2), U7.24 (PA13)
- new net UART_RX: R15.2, U7.21 (PA10/NC), U9.4
- new net UART_TX: U7.19 (PA9/NC), U8.2
- new net shunt+: NT1.1, R5.2, R7.1
Other:
- note removed: "Connect + and - in directly to shunt pads."
- moved on the sheet: C101, C12, C2, C3, C4, C5, C6, C7, C9, D2, D3, F1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
